File: rc2robot.kicad_pcb (KiCad board)
At the start: 2 copper layers, 28 x 29.4 mm, 14 parts, among them J1 Conn_01x06, J2 Conn_01x03, J3 Conn_Debug, J4 CAN_conn, U1 STM32F303K8Tx, U2 TCAN332, U3 LD1117S33TR_SOT223

Commit message: finish board
Parts:
- added C4: 1u, Capacitor_SMD:C_0805_2012Metric_Pad1.15x1.40mm_HandSolder, F.Cu at (107.8, 119.4)
- added J5: Conn_01x03, Connector_JST:JST_XH_B3B-XH-A_1x03_P2.50mm_Vertical, F.Cu at (125.8, 121.0)
- J3: footprint Connector_JST:JST_PH_B4B-PH-K_1x04_P2.00mm_Vertical -> Connector_JST:JST_PH_B6B-PH-K_1x06_P2.00mm_Vertical
- moved R2 10.9 mm to (112.8, 107.0)
- moved J4 8.98 mm to (125.8, 110.0)
- moved D1 7.20 mm to (108.8, 98.4)
- moved R1 7.20 mm to (108.8, 100.6)
- moved C3 7.16 mm to (121.6, 99.0), turned to 270 degrees
- moved U3 6.40 mm to (116.0, 100.2)
- moved U1 6.00 mm to (111.4, 113.2)
- moved J1 3.40 mm to (101.6, 111.0)
- moved C6 3.21 mm to (118.6, 105.0)
- moved J2 3.20 mm to (101.6, 105.4)
- moved C1 3.16 mm to (117.8, 117.8)
- moved C2 3.06 mm to (120.4, 117.8)
- moved U2 2.79 mm to (119.8, 112.0)
- moved J3 1.00 mm to (118.4, 123.8), turned to 180 degrees
Connections:
- J2 pad 3: /Bnd|Dat -> (no net)
- J4 pad 2: /CAN/CAN_NRST -> (no net)
- U1 pad 10: Net-(U1-Pad10) -> /Rudd
- U1 pad 11: Net-(U1-Pad11) -> (no net)
- U1 pad 12: Net-(U1-Pad12) -> /Gear
- U1 pad 13: Net-(U1-Pad13) -> (no net)
- U1 pad 14: Net-(U1-Pad14) -> (no net)
- U1 pad 15: Net-(U1-Pad15) -> (no net)
- U1 pad 18: Net-(U1-Pad18) -> /Aux1
- U1 pad 19: Net-(U1-Pad19) -> (no net)
- U1 pad 2: Net-(U1-Pad2) -> (no net)
- U1 pad 20: Net-(U1-Pad20) -> (no net)
- U1 pad 25: Net-(U1-Pad25) -> (no net)
- U1 pad 26: Net-(U1-Pad26) -> (no net)
- U1 pad 27: Net-(U1-Pad27) -> (no net)
- U1 pad 28: Net-(U1-Pad28) -> (no net)
- U1 pad 29: Net-(U1-Pad29) -> /USART1_TX
- U1 pad 3: Net-(U1-Pad3) -> (no net)
- U1 pad 30: Net-(U1-Pad30) -> /USART1_RX
- U1 pad 31: Net-(U1-Pad31) -> (no net)
- U1 pad 6: Net-(U1-Pad6) -> /Thro
- U1 pad 7: Net-(U1-Pad7) -> (no net)
- U1 pad 8: Net-(U1-Pad8) -> /Aile
- U1 pad 9: Net-(U1-Pad9) -> /Elev
- U2 pad 5: Net-(U2-Pad5) -> (no net)
- U2 pad 8: Net-(U2-Pad8) -> (no net)
Routing:
- net +3V3: track 14.6 -> 54.2 mm, vias 0 -> 3
- net /USART1_RX: track 0.00 -> 36.2 mm, vias 0 -> 2
- net /USART1_TX: track 0.00 -> 30.2 mm, vias 0 -> 2
- net GND: track 4.76 -> 24.4 mm
- net /~RST: track 0.00 -> 18.8 mm, vias 0 -> 2
- net /CAN_RX: track 0.00 -> 14.5 mm, vias 0 -> 2
- net /Aux1: track 0.00 -> 13.0 mm, vias 0 -> 2
- net /Thro: track 0.00 -> 10.8 mm
- net +7.5V: track 40.8 -> 31.0 mm
- net /CAN_TX: track 0.00 -> 9.40 mm, vias 0 -> 2
- net /Gear: track 0.00 -> 9.03 mm
- net /Aile: track 0.00 -> 8.65 mm
- net /Rudd: track 0.00 -> 8.63 mm
- net /Elev: track 0.00 -> 7.53 mm
- net /TMS: track 0.00 -> 6.84 mm
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Other:
- board size 28 x 29.4 mm -> 30 x 29.4 mm
